File: bedroom_lights.kicad_pcb (KiCad board)
At the start: 2 copper layers, 78 x 58 mm, 71 parts, among them J1 GT-USB-7010ASV, J10 From_E-stop, J11 From_E-stop, J2 Conn_01x05_Pin, J3 Conn_01x10_Pin, J4 From_E-stop, J5 694106301002, J6 From_E-stop, J7 From_E-stop, J8 From_E-stop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

Commit message: ERC
Connections:
- net /MCU/GPIO10 renamed /MCU/CSO1
- net /MCU/GPIO12 renamed /MCU/CSO2
- net /MCU/GPIO16 renamed /MCU/LSS2
- net /MCU/GPIO9 renamed /MCU/LSS1
Changed lines of the file:
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@@
 	(net 7 "/MCU/GPIO14")
 	(net 8 "/MCU/GPIO13")
-	(net 9 "/MCU/GPIO10")
+	(net 9 "/MCU/LSS1")
 	(net 10 "/MCU/GPIO15")
 	(net 11 "/MCU/CS0")
@@
 	(net 29 "/MCU/ADC")
 	(net 30 "/MCU/GPIO0")
-	(net 31 "/MCU/GPIO9")
+	(net 31 "/MCU/CSO2")
 	(net 32 "/USB/SHIELD")
 	(net 33 "/MCU/GPIO5")
-	(net 34 "/MCU/GPIO16")
+	(net 34 "/MCU/LSS2")
 	(net 35 "/MCU/EN")
-	(net 36 "/MCU/GPIO12")
+	(net 36 "/MCU/CSO1")
 	(net 37 "/USB/CP2104_~{RST}")
 	(net 38 "unconnected-(J1-SBU2-PadB8)")
@@
 			(layers "F.Cu" "F.Mask" "F.Paste")
 			(roundrect_rratio 0.243902)
-			(net 9 "/MCU/GPIO10")
+			(net 36 "/MCU/CSO1")
 			(pintype "passive")
 		)
@@
 			(size 2.5 1)
 			(layers "F.Cu" "F.Mask" "F.Paste")
-			(net 34 "/MCU/GPIO16")
+			(net 34 "/MCU/LSS2")
 			(pinfunction "GPIO16")
 			(pintype "bidirectional")
@@
 			(size 2.5 1)
 			(layers "F.Cu" "F.Mask" "F.Paste")
-			(net 36 "/MCU/GPIO12")
+			(net 31 "/MCU/CSO2")
 			(pinfunction "GPIO12")
 			(pintype "bidirectional")
@@
 			(size 1 1.8)
 			(layers "F.Cu" "F.Mask" "F.Paste")
-			(net 31 "/MCU/GPIO9")
+			(net 9 "/MCU/LSS1")
 			(pinfunction "GPIO9")
 			(pintype "bidirectional")
@@
 			(size 1 1.8)
 			(layers "F.Cu" "F.Mask" "F.Paste")
-			(net 9 "/MCU/GPIO10")
+			(net 36 "/MCU/CSO1")
 			(pinfunction "GPIO10")
 			(pintype "bidirectional")
@@
 			(layers "*.Cu" "*.Mask")
 			(remove_unused_layers no)
-			(net 9 "/MCU/GPIO10")
+			(net 36 "/MCU/CSO1")
 			(pinfunction "Pin_10")
 			(pintype "passive")
@@
 			(layers "*.Cu" "*.Mask")
 			(remove_unused_layers no)
-			(net 34 "/MCU/GPIO16")
+			(net 34 "/MCU/LSS2")
 			(pinfunction "Pin_4")
 			(pintype "passive")
@@
 			(layers "*.Cu" "*.Mask")
 			(remove_unused_layers no)
-			(net 36 "/MCU/GPIO12")
+			(net 31 "/MCU/CSO2")
 			(pinfunction "Pin_5")
 			(pintype "passive")
@@
 			(layers "*.Cu" "*.Mask")
 			(remove_unused_layers no)
-			(net 31 "/MCU/GPIO9")
+			(net 9 "/MCU/LSS1")
 			(pinfunction "Pin_12")
 			(pintype "passive")
@@
 			(layers "F.Cu" "F.Mask" "F.Paste")
 			(roundrect_rratio 0.243902)
-			(net 31 "/MCU/GPIO9")
+			(net 9 "/MCU/LSS1")
 			(pintype "passive")
 		)
@@
 			(layers "F.Cu" "F.Mask" "F.Paste")
 			(roundrect_rratio 0.243902)
-			(net 34 "/MCU/GPIO16")
+			(net 34 "/MCU/LSS2")
 			(pintype "passive")
 		)
@@
 			(layers "F.Cu" "F.Mask" "F.Paste")
 			(roundrect_rratio 0.243902)
-			(net 36 "/MCU/GPIO12")
+			(net 31 "/MCU/CSO2")
 			(pintype "passive")
 		)
@@
 	)
 	(segment
-		(start 153.5 94.5)
-		(end 158.01379 94.5)
-		(width 0.4)
-		(layer "F.Cu")
-		(net 9)
-	)
-	(segment
-		(start 151 70)
-		(end 151 75)
-		(width 0.4)
+		(start 131 89)
+		(end 136 84)
+		(width 0.3)
 		(layer "F.Cu")
 		(net 9)
 	)
 	(segment
-		(start 150.9125 96)
-		(end 152 96)
-		(width 0.4)
+		(start 136 84)
+		(end 136 83.62)
+		(width 0.3)
 		(layer "F.Cu")
 		(net 9)
 	)
 	(segment
-		(start 151 75)
-		(end 154.16 78.16)
-		(width 0.4)
+		(start 130.9125 89)
+		(end 131 89)
+		(width 0.3)
 		(layer "F.Cu")
 		(net 9)
 	)
 	(segment
-		(start 154.16 78.16)
-		(end 164 78.16)
+		(start 149 72)
+		(end 149 70)
 		(width 0.4)
 		(layer "F.Cu")
 		(net 9)
 	)
-	(segment
-		(start 159.5 78.16)
-		(end 164 78.16)
-		(width 0.4)
-		(layer "F.Cu")
+	(via
+		(at 149 72)
+		(size 0.8)
+		(drill 0.4)
+		(layers "F.Cu" "B.Cu")
 		(net 9)
 	)
 	(segment
-		(start 152 96)
-		(end 153.5 94.5)
+		(start 139.88 83.62)
+		(end 136 83.62)
 		(width 0.4)
-		(layer "F.Cu")
+		(layer "B.Cu")
 		(net 9)
 	)
 	(segment
-		(start 158.01379 94.5)
-		(end 159.5 93.01379)
+		(start 149 72)
+		(end 149 74.5)
 		(width 0.4)
-		(layer "F.Cu")
+		(layer "B.Cu")
 		(net 9)
 	)
 	(segment
-		(start 159.5 93.01379)
-		(end 159.5 78.16)
+		(start 149 74.5)
+		(end 139.88 83.62)
 		(width 0.4)
-		(layer "F.Cu")
+		(layer "B.Cu")
 		(net 9)
 	)
@@
 	)
 	(segment
-		(start 131 89)
-		(end 136 84)
-		(width 0.3)
+		(start 139.4125 96)
+		(end 138.3115 97.101)
+		(width 0.4)
 		(layer "F.Cu")
 		(net 31)
 	)
 	(segment
-		(start 136 84)
-		(end 136 83.62)
-		(width 0.3)
+		(start 138.3115 97.101)
+		(end 137.04842 97.101)
+		(width 0.4)
 		(layer "F.Cu")
 		(net 31)
 	)
 	(segment
-		(start 130.9125 89)
-		(end 131 89)
-		(width 0.3)
+		(start 136.501 96.009468)
+		(end 135.491532 95)
+		(width 0.4)
 		(layer "F.Cu")
 		(net 31)
 	)
 	(segment
-		(start 149 72)
-		(end 149 70)
+		(start 137.04842 97.101)
+		(end 136.501 96.55358)
+		(width 0.4)
+		(layer "F.Cu")
+		(net 31)
+	)
+	(segment
+		(start 142.4 64.5)
+		(end 137.34 64.5)
+		(width 0.4)
+		(layer "F.Cu")
+		(net 31)
+	)
+	(segment
+		(start 137.34 64.5)
+		(end 136 65.84)
+		(width 0.4)
+		(layer "F.Cu")
+		(net 31)
+	)
+	(segment
+		(start 135.491532 95)
+		(end 134.5 95)
+		(width 0.4)
+		(layer "F.Cu")
+		(net 31)
+	)
+	(segment
+		(start 136.501 96.55358)
+		(end 136.501 96.009468)
 		(width 0.4)
 		(layer "F.Cu")
@@
 	)
 	(via
-		(at 149 72)
+		(at 134.5 95)
 		(size 0.8)
 		(drill 0.4)
@@
 	)
 	(segment
-		(start 139.88 83.62)
-		(end 136 83.62)
+		(start 134.5 95)
+		(end 130.952 91.452)
 		(width 0.4)
 		(layer "B.Cu")
@@
 	)
 	(segment
-		(start 149 72)
-		(end 149 74.5)
+		(start 130.952 70.888)
+		(end 136 65.84)
 		(width 0.4)
 		(layer "B.Cu")
@@
 	)
 	(segment
-		(start 149 74.5)
-		(end 139.88 83.62)
+		(start 130.952 91.452)
+		(end 130.952 70.888)
 		(width 0.4)
 		(layer "B.Cu")
@@
 	)
 	(segment
-		(start 139.4125 96)
-		(end 138.3115 97.101)
+		(start 153.5 94.5)
+		(end 158.01379 94.5)
 		(width 0.4)
 		(layer "F.Cu")
@@
 	)
 	(segment
-		(start 138.3115 97.101)
-		(end 137.04842 97.101)
+		(start 151 70)
+		(end 151 75)
 		(width 0.4)
 		(layer "F.Cu")
@@
 	)
 	(segment
-		(start 136.501 96.009468)
-		(end 135.491532 95)
+		(start 150.9125 96)
+		(end 152 96)
 		(width 0.4)
 		(layer "F.Cu")
@@
 	)
 	(segment
-		(start 137.04842 97.101)
-		(end 136.501 96.55358)
+		(start 151 75)
+		(end 154.16 78.16)
 		(width 0.4)
 		(layer "F.Cu")
@@
 	)
 	(segment
-		(start 142.4 64.5)
-		(end 137.34 64.5)
+		(start 154.16 78.16)
+		(end 164 78.16)
 		(width 0.4)
 		(layer "F.Cu")
@@
 	)
 	(segment
-		(start 137.34 64.5)
-		(end 136 65.84)
+		(start 159.5 78.16)
+		(end 164 78.16)
 		(width 0.4)
 		(layer "F.Cu")
@@
 	)
 	(segment
-		(start 135.491532 95)
-		(end 134.5 95)
+		(start 152 96)
+		(end 153.5 94.5)
 		(width 0.4)
 		(layer "F.Cu")
@@
 	)
 	(segment
-		(start 136.501 96.55358)
-		(end 136.501 96.009468)
+		(start 158.01379 94.5)
+		(end 159.5 93.01379)
 		(width 0.4)
 		(layer "F.Cu")
 		(net 36)
 	)
-	(via
-		(at 134.5 95)
-		(size 0.8)
-		(drill 0.4)
-		(layers "F.Cu" "B.Cu")
-		(net 36)
-	)
-	(segment
-		(start 134.5 95)
-		(end 130.952 91.452)
-		(width 0.4)
-		(layer "B.Cu")
-		(net 36)
-	)
-	(segment
-		(start 130.952 70.888)
-		(end 136 65.84)
-		(width 0.4)
-		(layer "B.Cu")
-		(net 36)
-	)
 	(segment
-		(start 130.952 91.452)
-		(end 130.952 70.888)
+		(start 159.5 93.01379)
+		(end 159.5 78.16)
 		(width 0.4)
-		(layer "B.Cu")
+		(layer "F.Cu")
 		(net 36)
 	)
