File: epd.kicad_sch (KiCad schematic)
At the start: 19 parts, among them J4 FH12A-24S-0.5SH(55), Q3 Q_NMOS_GSD

Commit message: Renamifications
Parts:
- J4: symbol bedroom_lights:FPC24_Inverted -> lighthouse:FPC24_Inverted
- L1: footprint bedroom_lights:L_4x4x2.6 -> lighthouse:L_4x4x2.6
Changed lines of the file:
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@@
 		)
 		(instances
-			(project "bedroom_lights"
+			(project "lighthouse"
 				(path "/50da2b4e-34b1-4787-8ee6-5d7d17f804f4/d598949e-74c6-4803-8db9-612ef03f3111"
 					(reference "C15")
@@
 		)
 		(instances
-			(project "bedroom_lights"
+			(project "lighthouse"
 				(path "/50da2b4e-34b1-4787-8ee6-5d7d17f804f4/d598949e-74c6-4803-8db9-612ef03f3111"
 					(reference "#PWR018")
@@
 		)
 		(instances
-			(project "bedroom_lights"
+			(project "lighthouse"
 				(path "/50da2b4e-34b1-4787-8ee6-5d7d17f804f4/d598949e-74c6-4803-8db9-612ef03f3111"
 					(reference "#PWR030")
@@
 		)
 		(instances
-			(project "bedroom_lights"
+			(project "lighthouse"
 				(path "/50da2b4e-34b1-4787-8ee6-5d7d17f804f4/d598949e-74c6-4803-8db9-612ef03f3111"
 					(reference "#FLG05")
@@
 		)
 		(instances
-			(project "bedroom_lights"
+			(project "lighthouse"
 				(path "/50da2b4e-34b1-4787-8ee6-5d7d17f804f4/d598949e-74c6-4803-8db9-612ef03f3111"
 					(reference "C14")
@@
 		)
 		(instances
-			(project "bedroom_lights"
+			(project "lighthouse"
 				(path "/50da2b4e-34b1-4787-8ee6-5d7d17f804f4/d598949e-74c6-4803-8db9-612ef03f3111"
 					(reference "C8")
@@
 		)
 		(instances
-			(project "bedroom_lights"
+			(project "lighthouse"
 				(path "/50da2b4e-34b1-4787-8ee6-5d7d17f804f4/d598949e-74c6-4803-8db9-612ef03f3111"
 					(reference "#PWR027")
@@
 		)
 		(instances
-			(project "bedroom_lights"
+			(project "lighthouse"
 				(path "/50da2b4e-34b1-4787-8ee6-5d7d17f804f4/d598949e-74c6-4803-8db9-612ef03f3111"
 					(reference "#PWR020")
@@
 			)
 		)
-		(property "Footprint" "bedroom_lights:L_4x4x2.6"
+		(property "Footprint" "lighthouse:L_4x4x2.6"
 			(at 63.5 76.2 0)
 			(effects
@@
 		)
 		(instances
-			(project "bedroom_lights"
+			(project "lighthouse"
 				(path "/50da2b4e-34b1-4787-8ee6-5d7d17f804f4/d598949e-74c6-4803-8db9-612ef03f3111"
 					(reference "L1")
@@
 		)
 		(instances
-			(project "bedroom_lights"
+			(project "lighthouse"
 				(path "/50da2b4e-34b1-4787-8ee6-5d7d17f804f4/d598949e-74c6-4803-8db9-612ef03f3111"
 					(reference "D4")
@@
 		)
 		(instances
-			(project "bedroom_lights"
+			(project "lighthouse"
 				(path "/50da2b4e-34b1-4787-8ee6-5d7d17f804f4/d598949e-74c6-4803-8db9-612ef03f3111"
 					(reference "C13")
@@
 		)
 		(instances
-			(project "bedroom_lights"
+			(project "lighthouse"
 				(path "/50da2b4e-34b1-4787-8ee6-5d7d17f804f4/d598949e-74c6-4803-8db9-612ef03f3111"
 					(reference "D2")
@@
 		)
 		(instances
-			(project "bedroom_lights"
+			(project "lighthouse"
 				(path "/50da2b4e-34b1-4787-8ee6-5d7d17f804f4/d598949e-74c6-4803-8db9-612ef03f3111"
 					(reference "#PWR026")
@@
 		)
 		(instances
-			(project "bedroom_lights"
+			(project "lighthouse"
 				(path "/50da2b4e-34b1-4787-8ee6-5d7d17f804f4/d598949e-74c6-4803-8db9-612ef03f3111"
 					(reference "#PWR025")
@@
 		)
 		(instances
-			(project "bedroom_lights"
+			(project "lighthouse"
 				(path "/50da2b4e-34b1-4787-8ee6-5d7d17f804f4/d598949e-74c6-4803-8db9-612ef03f3111"
 					(reference "#PWR016")
@@
 		)
 		(instances
-			(project "bedroom_lights"
+			(project "lighthouse"
 				(path "/50da2b4e-34b1-4787-8ee6-5d7d17f804f4/d598949e-74c6-4803-8db9-612ef03f3111"
 					(reference "#PWR019")
@@
 		)
 		(instances
-			(project "bedroom_lights"
+			(project "lighthouse"
 				(path "/50da2b4e-34b1-4787-8ee6-5d7d17f804f4/d598949e-74c6-4803-8db9-612ef03f3111"
 					(reference "R13")
@@
 		)
 		(instances
-			(project "bedroom_lights"
+			(project "lighthouse"
 				(path "/50da2b4e-34b1-4787-8ee6-5d7d17f804f4/d598949e-74c6-4803-8db9-612ef03f3111"
 					(reference "C9")
@@
 		)
 		(instances
-			(project "bedroom_lights"
+			(project "lighthouse"
 				(path "/50da2b4e-34b1-4787-8ee6-5d7d17f804f4/d598949e-74c6-4803-8db9-612ef03f3111"
 					(reference "#PWR017")
@@
 		)
 		(instances
-			(project "bedroom_lights"
+			(project "lighthouse"
 				(path "/50da2b4e-34b1-4787-8ee6-5d7d17f804f4/d598949e-74c6-4803-8db9-612ef03f3111"
 					(reference "Q3")
@@
 		)
 		(instances
-			(project "bedroom_lights"
+			(project "lighthouse"
 				(path "/50da2b4e-34b1-4787-8ee6-5d7d17f804f4/d598949e-74c6-4803-8db9-612ef03f3111"
 					(reference "C16")
@@
 	)
 	(symbol
-		(lib_id "bedroom_lights:FPC24_Inverted")
+		(lib_id "lighthouse:FPC24_Inverted")
 		(at 255.27 85.09 0)
 		(unit 1)
@@
 		)
 		(instances
-			(project "bedroom_lights"
+			(project "lighthouse"
 				(path "/50da2b4e-34b1-4787-8ee6-5d7d17f804f4/d598949e-74c6-4803-8db9-612ef03f3111"
 					(reference "J4")
@@
 		)
 		(instances
-			(project "bedroom_lights"
+			(project "lighthouse"
 				(path "/50da2b4e-34b1-4787-8ee6-5d7d17f804f4/d598949e-74c6-4803-8db9-612ef03f3111"
 					(reference "#PWR029")
@@
 		)
 		(instances
-			(project "bedroom_lights"
+			(project "lighthouse"
 				(path "/50da2b4e-34b1-4787-8ee6-5d7d17f804f4/d598949e-74c6-4803-8db9-612ef03f3111"
 					(reference "C18")
@@
 		)
 		(instances
-			(project "bedroom_lights"
+			(project "lighthouse"
 				(path "/50da2b4e-34b1-4787-8ee6-5d7d17f804f4/d598949e-74c6-4803-8db9-612ef03f3111"
 					(reference "#FLG04")
@@
 		)
 		(instances
-			(project "bedroom_lights"
+			(project "lighthouse"
 				(path "/50da2b4e-34b1-4787-8ee6-5d7d17f804f4/d598949e-74c6-4803-8db9-612ef03f3111"
 					(reference "#PWR024")
@@
 		)
 		(instances
-			(project "bedroom_lights"
+			(project "lighthouse"
 				(path "/50da2b4e-34b1-4787-8ee6-5d7d17f804f4/d598949e-74c6-4803-8db9-612ef03f3111"
 					(reference "#PWR021")
@@
 		)
 		(instances
-			(project "bedroom_lights"
+			(project "lighthouse"
 				(path "/50da2b4e-34b1-4787-8ee6-5d7d17f804f4/d598949e-74c6-4803-8db9-612ef03f3111"
 					(reference "#PWR022")
@@
 		)
 		(instances
-			(project "bedroom_lights"
+			(project "lighthouse"
 				(path "/50da2b4e-34b1-4787-8ee6-5d7d17f804f4/d598949e-74c6-4803-8db9-612ef03f3111"
 					(reference "R12")
@@
 		)
 		(instances
-			(project "bedroom_lights"
+			(project "lighthouse"
 				(path "/50da2b4e-34b1-4787-8ee6-5d7d17f804f4/d598949e-74c6-4803-8db9-612ef03f3111"
 					(reference "#PWR028")
@@
 		)
 		(instances
-			(project "bedroom_lights"
+			(project "lighthouse"
 				(path "/50da2b4e-34b1-4787-8ee6-5d7d17f804f4/d598949e-74c6-4803-8db9-612ef03f3111"
 					(reference "D3")
@@
 		)
 		(instances
-			(project "bedroom_lights"
+			(project "lighthouse"
 				(path "/50da2b4e-34b1-4787-8ee6-5d7d17f804f4/d598949e-74c6-4803-8db9-612ef03f3111"
 					(reference "C12")
@@
 		)
 		(instances
-			(project "bedroom_lights"
+			(project "lighthouse"
 				(path "/50da2b4e-34b1-4787-8ee6-5d7d17f804f4/d598949e-74c6-4803-8db9-612ef03f3111"
 					(reference "C10")
@@
 		)
 		(instances
-			(project "bedroom_lights"
+			(project "lighthouse"
 				(path "/50da2b4e-34b1-4787-8ee6-5d7d17f804f4/d598949e-74c6-4803-8db9-612ef03f3111"
 					(reference "C17")
@@
 		)
 		(instances
-			(project "bedroom_lights"
+			(project "lighthouse"
 				(path "/50da2b4e-34b1-4787-8ee6-5d7d17f804f4/d598949e-74c6-4803-8db9-612ef03f3111"
 					(reference "C11")
@@
 		)
 		(instances
-			(project "bedroom_lights"
+			(project "lighthouse"
 				(path "/50da2b4e-34b1-4787-8ee6-5d7d17f804f4/d598949e-74c6-4803-8db9-612ef03f3111"
 					(reference "#PWR023")
