File: low_side_switch.kicad_sch (KiCad schematic)
At the start: 7 parts, among them J8 From_E-stop, J9 From_E-stop, Q7 S8050, Q8 BSS138-7-F

Commit message: Termianl block 3d view
Parts:
- J8, J9: value From_E-stop -> TB0010-500-02GR; footprint TerminalBlock:TerminalBlock_MaiXu_MX126-5.0-02P_1x02_P5.00mm -> lighthouse:TerminalBlock_TB0010-500-02GR_1x02_P5.00mm
Changed lines of the file:
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@@
 			)
 		)
-		(property "Value" "From_E-stop"
+		(property "Value" "TB0010-500-02GR"
 			(at 35.56 44.45 0)
 			(effects
@@
 			)
 		)
-		(property "Footprint" "TerminalBlock:TerminalBlock_MaiXu_MX126-5.0-02P_1x02_P5.00mm"
+		(property "Footprint" "lighthouse:TerminalBlock_TB0010-500-02GR_1x02_P5.00mm"
 			(at 35.56 48.26 0)
 			(effects
@@
 			)
 		)
-		(property "Value" "From_E-stop"
+		(property "Value" "TB0010-500-02GR"
 			(at 116.84 44.45 0)
 			(effects
@@
 			)
 		)
-		(property "Footprint" "TerminalBlock:TerminalBlock_MaiXu_MX126-5.0-02P_1x02_P5.00mm"
+		(property "Footprint" "lighthouse:TerminalBlock_TB0010-500-02GR_1x02_P5.00mm"
 			(at 116.84 48.26 0)
 			(effects

Commit message: Add component attributes
Parts:
- Q7: value S8050 -> MMSS8050-H-TP
- R18: MPN (none) -> CRCW0805220RJNEA; Manufacturer (none) -> Vishay; Mouser Part Number (none) -> 71-CRCW0805220RJNEA; Package (none) -> 0805
- R19: MPN (none) -> CRCW080510K0JNEAC; Manufacturer (none) -> Vishay; Mouser Part Number (none) -> 71-CRCW080510K0JNEAC; Package (none) -> 0805; Power (none) -> 125mW; Tolerance (none) -> 5 %
Changed lines of the file:
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@@
+			)
+		)
+		(property "Manufactuer" ""
+			(at 101.6 63.5 0)
+			(effects
+				(font
+					(size 1.27 1.27)
+				)
+				(hide yes)
 			)
 		)
@@
 			)
 		)
+		(property "Manufactuer" ""
+			(at 50.8 40.64 0)
+			(effects
+				(font
+					(size 1.27 1.27)
+				)
+				(hide yes)
+			)
+		)
 		(pin "3"
 		)
@@
 			)
 		)
+		(property "Manufactuer" ""
+			(at 35.56 48.26 0)
+			(effects
+				(font
+					(size 1.27 1.27)
+				)
+				(hide yes)
+			)
+		)
 		(pin "1"
 		)
@@
 			)
 		)
+		(property "LCSC Part Number" ""
+			(at 86.36 55.88 0)
+			(effects
+				(font
+					(size 1.27 1.27)
+				)
+				(hide yes)
+			)
+		)
+		(property "MPN" "CRCW080510K0JNEAC"
+			(at 86.36 55.88 0)
+			(effects
+				(font
+					(size 1.27 1.27)
+				)
+				(hide yes)
+			)
+		)
+		(property "Manufacturer" "Vishay "
+			(at 86.36 55.88 0)
+			(effects
+				(font
+					(size 1.27 1.27)
+				)
+				(hide yes)
+			)
+		)
+		(property "Package" "0805"
+			(at 86.36 55.88 0)
+			(effects
+				(font
+					(size 1.27 1.27)
+				)
+				(hide yes)
+			)
+		)
+		(property "Power" "125mW"
+			(at 86.36 55.88 0)
+			(effects
+				(font
+					(size 1.27 1.27)
+				)
+				(hide yes)
+			)
+		)
+		(property "Tolerance" "5 %"
+			(at 86.36 55.88 0)
+			(effects
+				(font
+					(size 1.27 1.27)
+				)
+				(hide yes)
+			)
+		)
+		(property "Manufactuer" ""
+			(at 86.36 55.88 0)
+			(effects
+				(font
+					(size 1.27 1.27)
+				)
+				(hide yes)
+			)
+		)
+		(property "Mouser Part Number" "71-CRCW080510K0JNEAC"
+			(at 86.36 55.88 0)
+			(effects
+				(font
+					(size 1.27 1.27)
+				)
+				(hide yes)
+			)
+		)
 		(pin "2"
 		)
@@
 			)
 		)
+		(property "MPN" "CRCW0805220RJNEA "
+			(at 66.04 76.2 90)
+			(effects
+				(font
+					(size 1.27 1.27)
+				)
+				(hide yes)
+			)
+		)
+		(property "Manufacturer" "Vishay "
+			(at 66.04 76.2 90)
+			(effects
+				(font
+					(size 1.27 1.27)
+				)
+				(hide yes)
+			)
+		)
+		(property "Mouser Part Number" "71-CRCW0805220RJNEA "
+			(at 66.04 76.2 90)
+			(effects
+				(font
+					(size 1.27 1.27)
+				)
+				(hide yes)
+			)
+		)
+		(property "Package" "0805"
+			(at 66.04 76.2 90)
+			(effects
+				(font
+					(size 1.27 1.27)
+				)
+				(hide yes)
+			)
+		)
+		(property "Manufactuer" ""
+			(at 66.04 76.2 90)
+			(effects
+				(font
+					(size 1.27 1.27)
+				)
+				(hide yes)
+			)
+		)
 		(pin "1"
 		)
@@
 		)
 		(property "Description" "Generic screw terminal, single row, 01x02, script generated (kicad-library-utils/schlib/autogen/connector/)"
+			(at 116.84 48.26 0)
+			(effects
+				(font
+					(size 1.27 1.27)
+				)
+				(hide yes)
+			)
+		)
+		(property "Manufactuer" ""
 			(at 116.84 48.26 0)
 			(effects
@@
 			)
 		)
-		(property "Value" "S8050"
+		(property "Value" "MMSS8050-H-TP"
 			(at 88.9 77.4699 0)
 			(effects
@@
 			(at 83.82 76.2 0)
 			(effects
+				(font
+					(size 1.27 1.27)
+				)
+				(hide yes)
+			)
+		)
+		(property "Manufactuer" ""
+			(at 83.82 76.2 0)
+			(effects
