File: usb.kicad_sch (KiCad schematic)
At the start: 14 parts, among them J1 GT-USB-7010ASV, Q1 S8050, Q2 S8050, U1 CP2104

Commit message: Lighthouse
Parts:
- J1: footprint youdbetterrun:USB_C_Receptacle_G-Switch_GT-USB-7010ASV -> bedroom_lights:USB_C_Receptacle_G-Switch_GT-USB-7010ASV
Other:
- company: (none) -> Marcel Robitaille
- title: (none) -> USB
Changed lines of the file:
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@@
 	(generator_version "9.0")
 	(paper "A4")
+	(title_block
+		(title "USB")
+		(date "2025-11-02")
+		(company "Marcel Robitaille")
+	)
 	(text "Place near VDD"
 		(exclude_from_sim no)
@@
 	)
 	(junction
-		(at 50.8 100.33)
-		(diameter 0)
-		(color 0 0 0 0)
-	)
-	(junction
 		(at 119.38 76.2)
 		(diameter 0)
@@
 	(wire
 		(pts
-			(xy 50.8 99.06) (xy 50.8 100.33)
+			(xy 50.8 99.06) (xy 50.8 101.6)
 		)
 		(stroke
@@
 	(wire
 		(pts
-			(xy 50.8 100.33) (xy 50.8 101.6)
-		)
-		(stroke
-			(width 0)
-			(type default)
-		)
-	)
-	(wire
-		(pts
 			(xy 119.38 76.2) (xy 162.56 76.2)
 		)
@@
 	)
 	(symbol
-		(lib_id "power:PWR_FLAG")
-		(at 50.8 100.33 270)
-		(unit 1)
-		(exclude_from_sim no)
-		(in_bom yes)
-		(on_board yes)
-		(dnp no)
-		(fields_autoplaced yes)
-		(property "Reference" "#FLG01"
-			(at 52.705 100.33 0)
-			(effects
-				(font
-					(size 1.27 1.27)
-				)
-				(hide yes)
-			)
-		)
-		(property "Value" "PWR_FLAG"
-			(at 54.61 100.3299 90)
-			(effects
-				(font
-					(size 1.27 1.27)
-				)
-				(justify left)
-			)
-		)
-		(property "Footprint" ""
-			(at 50.8 100.33 0)
-			(effects
-				(font
-					(size 1.27 1.27)
-				)
-				(hide yes)
-			)
-		)
-		(property "Datasheet" "~"
-			(at 50.8 100.33 0)
-			(effects
-				(font
-					(size 1.27 1.27)
-				)
-				(hide yes)
-			)
-		)
-		(property "Description" "Special symbol for telling ERC where power comes from"
-			(at 50.8 100.33 0)
-			(effects
-				(font
-					(size 1.27 1.27)
-				)
-				(hide yes)
-			)
-		)
-		(pin "1"
-		)
-		(instances
-			(project "youdbetterrun"
-				(path "/50da2b4e-34b1-4787-8ee6-5d7d17f804f4/951b5697-f1e3-4d2e-841e-7032f41eb35f"
-					(reference "#FLG01")
-					(unit 1)
-				)
-			)
-		)
-	)
-	(symbol
 		(lib_id "Connector:USB_C_Receptacle_USB2.0_16P")
 		(at 50.8 76.2 0)
@@
 			)
 		)
-		(property "Footprint" "youdbetterrun:USB_C_Receptacle_G-Switch_GT-USB-7010ASV"
+		(property "Footprint" "bedroom_lights:USB_C_Receptacle_G-Switch_GT-USB-7010ASV"
 			(at 54.61 76.2 0)
 			(effects
@@
 		)
 		(instances
-			(project "youdbetterrun"
+			(project "bedroom_lights"
 				(path "/50da2b4e-34b1-4787-8ee6-5d7d17f804f4/951b5697-f1e3-4d2e-841e-7032f41eb35f"
 					(reference "J1")
@@
 			)
 		)
-		(property "Datasheet" "https://www.lcsc.com/datasheet/C2891804.pdf"
+		(property "Datasheet" "~"
 			(at 256.54 119.38 0)
 			(effects
@@
 			)
 		)
-		(property "Description" "Bipolar (BJT) Transistor NPN 25 V 500 mA 150MHz 300 mW Surface Mount SOT-23"
+		(property "Description" "NPN transistor, base/emitter/collector"
 			(at 256.54 119.38 0)
 			(effects
@@
 		)
 		(instances
-			(project "youdbetterrun"
+			(project "bedroom_lights"
 				(path "/50da2b4e-34b1-4787-8ee6-5d7d17f804f4/951b5697-f1e3-4d2e-841e-7032f41eb35f"
 					(reference "Q2")
@@
 		)
 		(instances
-			(project "youdbetterrun"
+			(project "bedroom_lights"
 				(path "/50da2b4e-34b1-4787-8ee6-5d7d17f804f4/951b5697-f1e3-4d2e-841e-7032f41eb35f"
 					(reference "R2")
@@
 		)
 		(instances
-			(project "youdbetterrun"
+			(project "bedroom_lights"
 				(path "/50da2b4e-34b1-4787-8ee6-5d7d17f804f4/951b5697-f1e3-4d2e-841e-7032f41eb35f"
 					(reference "#FLG03")
@@
 		)
 		(instances
-			(project "youdbetterrun"
+			(project "bedroom_lights"
 				(path "/50da2b4e-34b1-4787-8ee6-5d7d17f804f4/951b5697-f1e3-4d2e-841e-7032f41eb35f"
 					(reference "#PWR08")
@@
 		)
 		(instances
-			(project "youdbetterrun"
+			(project "bedroom_lights"
 				(path "/50da2b4e-34b1-4787-8ee6-5d7d17f804f4/951b5697-f1e3-4d2e-841e-7032f41eb35f"
 					(reference "#PWR01")
@@
 		)
 		(instances
-			(project "youdbetterrun"
+			(project "bedroom_lights"
 				(path "/50da2b4e-34b1-4787-8ee6-5d7d17f804f4/951b5697-f1e3-4d2e-841e-7032f41eb35f"
 					(reference "C3")
@@
 		)
 		(instances
-			(project "youdbetterrun"
+			(project "bedroom_lights"
 				(path "/50da2b4e-34b1-4787-8ee6-5d7d17f804f4/951b5697-f1e3-4d2e-841e-7032f41eb35f"
 					(reference "#PWR06")
@@
 			)
 		)
-		(property "Datasheet" "https://datasheet.lcsc.com/lcsc/2206010200_UNI-ROYAL-Uniroyal-Elec-0805W8F4701T5E_C17673.pdf?_gl=1*1lzo6cr*_ga*MTgzMjI1NTEzNy4xNjg1MTA3NDAx*_ga_98M84MKSZH*MTcxNTQ0MDg0My4xMS4xLjE3MTU0NDEwMjIuNTcuMC4w"
+		(property "Datasheet" "~"
 			(at 160.02 43.18 0)
 			(effects
@@
 		)
 		(instances
-			(project "youdbetterrun"
+			(project "bedroom_lights"
 				(path "/50da2b4e-34b1-4787-8ee6-5d7d17f804f4/951b5697-f1e3-4d2e-841e-7032f41eb35f"
 					(reference "R3")
@@
 		)
 		(instances
-			(project "youdbetterrun"
+			(project "bedroom_lights"
 				(path "/50da2b4e-34b1-4787-8ee6-5d7d17f804f4/951b5697-f1e3-4d2e-841e-7032f41eb35f"
 					(reference "R4")
@@
 		)
 		(instances
-			(project "youdbetterrun"
+			(project "bedroom_lights"
 				(path "/50da2b4e-34b1-4787-8ee6-5d7d17f804f4/951b5697-f1e3-4d2e-841e-7032f41eb35f"
 					(reference "#PWR07")
@@
 		)
 		(instances
-			(project "youdbetterrun"
+			(project "bedroom_lights"
 				(path "/50da2b4e-34b1-4787-8ee6-5d7d17f804f4/951b5697-f1e3-4d2e-841e-7032f41eb35f"
 					(reference "C4")
@@
 		)
 		(instances
-			(project "youdbetterrun"
+			(project "bedroom_lights"
 				(path "/50da2b4e-34b1-4787-8ee6-5d7d17f804f4/951b5697-f1e3-4d2e-841e-7032f41eb35f"
 					(reference "C1")
@@
 		)
 		(instances
-			(project "youdbetterrun"
+			(project "bedroom_lights"
 				(path "/50da2b4e-34b1-4787-8ee6-5d7d17f804f4/951b5697-f1e3-4d2e-841e-7032f41eb35f"
 					(reference "U1")
@@
 		)
 		(instances
-			(project "youdbetterrun"
+			(project "bedroom_lights"
 				(path "/50da2b4e-34b1-4787-8ee6-5d7d17f804f4/951b5697-f1e3-4d2e-841e-7032f41eb35f"
 					(reference "R5")
@@
 		)
 		(instances
-			(project "youdbetterrun"
+			(project "bedroom_lights"
 				(path "/50da2b4e-34b1-4787-8ee6-5d7d17f804f4/951b5697-f1e3-4d2e-841e-7032f41eb35f"
 					(reference "D1")
@@
 		)
 		(instances
-			(project "youdbetterrun"
+			(project "bedroom_lights"
 				(path "/50da2b4e-34b1-4787-8ee6-5d7d17f804f4/951b5697-f1e3-4d2e-841e-7032f41eb35f"
 					(reference "R1")
@@
 		)
 		(instances
-			(project "youdbetterrun"
+			(project "bedroom_lights"
 				(path "/50da2b4e-34b1-4787-8ee6-5d7d17f804f4/951b5697-f1e3-4d2e-841e-7032f41eb35f"
 					(reference "#FLG02")
@@
 		)
 		(instances
-			(project "youdbetterrun"
+			(project "bedroom_lights"
 				(path "/50da2b4e-34b1-4787-8ee6-5d7d17f804f4/951b5697-f1e3-4d2e-841e-7032f41eb35f"
 					(reference "#PWR05")
@@
 		)
 		(instances
-			(project "youdbetterrun"
+			(project "bedroom_lights"
 				(path "/50da2b4e-34b1-4787-8ee6-5d7d17f804f4/951b5697-f1e3-4d2e-841e-7032f41eb35f"
 					(reference "C2")
@@
 		)
 		(instances
-			(project "youdbetterrun"
+			(project "bedroom_lights"
 				(path "/50da2b4e-34b1-4787-8ee6-5d7d17f804f4/951b5697-f1e3-4d2e-841e-7032f41eb35f"
 					(reference "#PWR03")
@@
 			)
 		)
-		(property "Datasheet" "https://www.lcsc.com/datasheet/C2891804.pdf"
+		(property "Datasheet" "~"
 			(at 256.54 93.98 0)
 			(effects
@@
 			)
 		)
-		(property "Description" "Bipolar (BJT) Transistor NPN 25 V 500 mA 150MHz 300 mW Surface Mount SOT-23"
+		(property "Description" "NPN transistor, base/emitter/collector"
 			(at 256.54 93.98 0)
 			(effects
@@
 		)
 		(instances
-			(project "youdbetterrun"
+			(project "bedroom_lights"
 				(path "/50da2b4e-34b1-4787-8ee6-5d7d17f804f4/951b5697-f1e3-4d2e-841e-7032f41eb35f"
 					(reference "Q1")
@@
 		)
 		(instances
-			(project "youdbetterrun"
+			(project "bedroom_lights"
 				(path "/50da2b4e-34b1-4787-8ee6-5d7d17f804f4/951b5697-f1e3-4d2e-841e-7032f41eb35f"
 					(reference "#PWR04")
@@
 		)
 		(instances
-			(project "youdbetterrun"
+			(project "bedroom_lights"
 				(path "/50da2b4e-34b1-4787-8ee6-5d7d17f804f4/951b5697-f1e3-4d2e-841e-7032f41eb35f"
 					(reference "#PWR02")

Commit message: ERC
Changed lines of the file:
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@@
 	)
 	(junction
+		(at 50.8 100.33)
+		(diameter 0)
+		(color 0 0 0 0)
+	)
+	(junction
 		(at 71.12 50.8)
 		(diameter 0)
@@
 	(wire
 		(pts
-			(xy 50.8 99.06) (xy 50.8 101.6)
+			(xy 50.8 99.06) (xy 50.8 100.33)
 		)
 		(stroke
@@
 	(wire
 		(pts
+			(xy 50.8 100.33) (xy 50.8 101.6)
+		)
+		(stroke
+			(width 0)
+			(type default)
+		)
+	)
+	(wire
+		(pts
 			(xy 43.18 111.76) (xy 121.92 111.76)
 		)
@@
 					(unit 1)
 				)
+			)
+		)
+	)
+	(symbol
+		(lib_id "power:PWR_FLAG")
+		(at 50.8 100.33 270)
+		(unit 1)
+		(exclude_from_sim no)
+		(in_bom yes)
+		(on_board yes)
+		(dnp no)
+		(fields_autoplaced yes)
+		(property "Reference" "#FLG01"
+			(at 52.705 100.33 0)
+			(effects
+				(font
+					(size 1.27 1.27)
+				)
+				(hide yes)
+			)
+		)
+		(property "Value" "PWR_FLAG"
+			(at 54.61 100.3299 90)
+			(effects
+				(font
+					(size 1.27 1.27)
+				)
+				(justify left)
+			)
+		)
+		(property "Footprint" ""
+			(at 50.8 100.33 0)
+			(effects
+				(font
+					(size 1.27 1.27)
+				)
+				(hide yes)
+			)
+		)
+		(property "Datasheet" "~"
+			(at 50.8 100.33 0)
+			(effects
+				(font
+					(size 1.27 1.27)
+				)
+				(hide yes)
+			)
+		)
+		(property "Description" "Special symbol for telling ERC where power comes from"
+			(at 50.8 100.33 0)
+			(effects
+				(font
+					(size 1.27 1.27)
+				)
+				(hide yes)
+			)
+		)
+		(pin "1"
+		)
+		(instances
+			(project ""
+				(path "/50da2b4e-34b1-4787-8ee6-5d7d17f804f4/951b5697-f1e3-4d2e-841e-7032f41eb35f"
+					(reference "#FLG01")
+					(unit 1)
+				)

Commit message: Renamifications
Parts:
- J1: footprint bedroom_lights:USB_C_Receptacle_G-Switch_GT-USB-7010ASV -> lighthouse:USB_C_Receptacle_G-Switch_GT-USB-7010ASV
Changed lines of the file:
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@@
 			)
 		)
-		(property "Footprint" "bedroom_lights:USB_C_Receptacle_G-Switch_GT-USB-7010ASV"
+		(property "Footprint" "lighthouse:USB_C_Receptacle_G-Switch_GT-USB-7010ASV"
 			(at 54.61 76.2 0)
 			(effects
@@
 		)
 		(instances
-			(project "bedroom_lights"
+			(project "lighthouse"
 				(path "/50da2b4e-34b1-4787-8ee6-5d7d17f804f4/951b5697-f1e3-4d2e-841e-7032f41eb35f"
 					(reference "J1")
@@
 		)
 		(instances
-			(project "bedroom_lights"
+			(project "lighthouse"
 				(path "/50da2b4e-34b1-4787-8ee6-5d7d17f804f4/951b5697-f1e3-4d2e-841e-7032f41eb35f"
 					(reference "Q2")
@@
 		)
 		(instances
-			(project "bedroom_lights"
+			(project "lighthouse"
 				(path "/50da2b4e-34b1-4787-8ee6-5d7d17f804f4/951b5697-f1e3-4d2e-841e-7032f41eb35f"
 					(reference "R2")
@@
 		)
 		(instances
-			(project "bedroom_lights"
+			(project "lighthouse"
 				(path "/50da2b4e-34b1-4787-8ee6-5d7d17f804f4/951b5697-f1e3-4d2e-841e-7032f41eb35f"
 					(reference "#FLG03")
@@
 		)
 		(instances
-			(project "bedroom_lights"
+			(project "lighthouse"
 				(path "/50da2b4e-34b1-4787-8ee6-5d7d17f804f4/951b5697-f1e3-4d2e-841e-7032f41eb35f"
 					(reference "#PWR08")
@@
 		)
 		(instances
-			(project "bedroom_lights"
+			(project "lighthouse"
 				(path "/50da2b4e-34b1-4787-8ee6-5d7d17f804f4/951b5697-f1e3-4d2e-841e-7032f41eb35f"
 					(reference "#PWR01")
@@
 		)
 		(instances
-			(project "bedroom_lights"
+			(project "lighthouse"
 				(path "/50da2b4e-34b1-4787-8ee6-5d7d17f804f4/951b5697-f1e3-4d2e-841e-7032f41eb35f"
 					(reference "C3")
@@
 		)
 		(instances
-			(project "bedroom_lights"
+			(project "lighthouse"
 				(path "/50da2b4e-34b1-4787-8ee6-5d7d17f804f4/951b5697-f1e3-4d2e-841e-7032f41eb35f"
 					(reference "#PWR06")
@@
 		)
 		(instances
-			(project "bedroom_lights"
+			(project "lighthouse"
 				(path "/50da2b4e-34b1-4787-8ee6-5d7d17f804f4/951b5697-f1e3-4d2e-841e-7032f41eb35f"
 					(reference "R3")
@@
 		)
 		(instances
-			(project "bedroom_lights"
+			(project "lighthouse"
 				(path "/50da2b4e-34b1-4787-8ee6-5d7d17f804f4/951b5697-f1e3-4d2e-841e-7032f41eb35f"
 					(reference "R4")
@@
 		)
 		(instances
-			(project "bedroom_lights"
+			(project "lighthouse"
 				(path "/50da2b4e-34b1-4787-8ee6-5d7d17f804f4/951b5697-f1e3-4d2e-841e-7032f41eb35f"
 					(reference "#PWR07")
@@
 		)
 		(instances
-			(project "bedroom_lights"
+			(project "lighthouse"
 				(path "/50da2b4e-34b1-4787-8ee6-5d7d17f804f4/951b5697-f1e3-4d2e-841e-7032f41eb35f"
 					(reference "C4")
@@
 		)
 		(instances
-			(project "bedroom_lights"
+			(project "lighthouse"
 				(path "/50da2b4e-34b1-4787-8ee6-5d7d17f804f4/951b5697-f1e3-4d2e-841e-7032f41eb35f"
 					(reference "C1")
@@
 		)
 		(instances
-			(project "bedroom_lights"
+			(project "lighthouse"
 				(path "/50da2b4e-34b1-4787-8ee6-5d7d17f804f4/951b5697-f1e3-4d2e-841e-7032f41eb35f"
 					(reference "U1")
@@
 		)
 		(instances
-			(project "bedroom_lights"
+			(project "lighthouse"
 				(path "/50da2b4e-34b1-4787-8ee6-5d7d17f804f4/951b5697-f1e3-4d2e-841e-7032f41eb35f"
 					(reference "R5")
@@
 		)
 		(instances
-			(project "bedroom_lights"
+			(project "lighthouse"
 				(path "/50da2b4e-34b1-4787-8ee6-5d7d17f804f4/951b5697-f1e3-4d2e-841e-7032f41eb35f"
 					(reference "D1")
@@
 		)
 		(instances
-			(project "bedroom_lights"
+			(project "lighthouse"
 				(path "/50da2b4e-34b1-4787-8ee6-5d7d17f804f4/951b5697-f1e3-4d2e-841e-7032f41eb35f"
 					(reference "R1")
@@
 		)
 		(instances
-			(project "bedroom_lights"
+			(project "lighthouse"
 				(path "/50da2b4e-34b1-4787-8ee6-5d7d17f804f4/951b5697-f1e3-4d2e-841e-7032f41eb35f"
 					(reference "#FLG02")
@@
 		)
 		(instances
-			(project "bedroom_lights"
+			(project "lighthouse"
 				(path "/50da2b4e-34b1-4787-8ee6-5d7d17f804f4/951b5697-f1e3-4d2e-841e-7032f41eb35f"
 					(reference "#PWR05")
@@
 		)
 		(instances
-			(project "bedroom_lights"
+			(project "lighthouse"
 				(path "/50da2b4e-34b1-4787-8ee6-5d7d17f804f4/951b5697-f1e3-4d2e-841e-7032f41eb35f"
 					(reference "C2")
@@
 		)
 		(instances
-			(project "bedroom_lights"
+			(project "lighthouse"
 				(path "/50da2b4e-34b1-4787-8ee6-5d7d17f804f4/951b5697-f1e3-4d2e-841e-7032f41eb35f"
 					(reference "#PWR03")
@@
 		)
 		(instances
-			(project "bedroom_lights"
+			(project "lighthouse"
 				(path "/50da2b4e-34b1-4787-8ee6-5d7d17f804f4/951b5697-f1e3-4d2e-841e-7032f41eb35f"
 					(reference "Q1")
@@
 		)
 		(instances
-			(project "bedroom_lights"
+			(project "lighthouse"
 				(path "/50da2b4e-34b1-4787-8ee6-5d7d17f804f4/951b5697-f1e3-4d2e-841e-7032f41eb35f"
 					(reference "#PWR04")
@@
 		)
 		(instances
-			(project "bedroom_lights"
+			(project "lighthouse"
 				(path "/50da2b4e-34b1-4787-8ee6-5d7d17f804f4/951b5697-f1e3-4d2e-841e-7032f41eb35f"
 					(reference "#PWR02")

Commit message: Add component attributes
Parts:
- Q1, Q2: LCSC Part Number C2891804 -> (none); MPN S8050 -> MMSS8050-L-TP; Manufacturer YONGYUTAI -> Micro Commercial Components (MCC); Mouser Part Number (none) -> 833-MMSS8050-L-TP
- R1, R2: LCSC Part Number C27834 -> (none); MPN 0805W8F5101T5E -> CRCW08055K10FKEAC; Manufacturer UNI-ROYAL(Uniroyal Elec) -> Vishay; Mouser Part Number (none) -> 71-CRCW08055K10FKEAC
- R3: LCSC Part Number C17673 -> (none); MPN 0805W8F4701T5E -> CR0805-FX-4701ELF; Manufacturer UNI-ROYAL(Uniroyal Elec) -> Bourns; Mouser Part Number (none) -> 652-CR0805FX-4701ELF; Package (none) -> 0805; Power (none) -> 125 mW; Tolerance (none) -> 1%
- R4, R5: LCSC Part Number C17444 -> (none); MPN 0805W8F1202T5E -> CRCW080512K0JNEA; Manufacturer UNI-ROYAL(Uniroyal Elec) -> Vishay; Mouser Part Number (none) -> 71-CRCW080512K0JNEA
